File: ergogen/output/pcbs/ergogen_footprints_demo.kicad_pcb (KiCad board)
At the start: 2 copper layers, 230 x 95 mm, 112 parts

Commit message: Update footprints library and add copper fill zone
Routing:
- added copper zone on F.Cu, net GND
Changed lines of the file:
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@@
     (segment (start 233.730 110.800) (end 233.730 112.550) (width 0.25) (layer "B.Cu") (net 99))
     (segment (start 231.190 110.800) (end 231.190 112.550) (width 0.25) (layer "B.Cu") (net 98))
+    (zone
+      (net 23)
+      (net_name "GND")
+      (locked no)
+      (layers "F.Cu")
+      (hatch edge 0.5)
+      (connect_pads
+        (clearance 0.508)
+      )
+      (min_thickness 0.25)
+      (filled_areas_thickness no)
+      (fill yes
+        (thermal_gap 0.5)
+        (thermal_bridge_width 0.5)
+        (smoothing chamfer)
+        (radius 0.5)
+        (island_removal_mode 1)
+        (island_area_min 5)
+      )
+      (polygon
+        (pts
+          (xy 0 0) (xy 420 0) (xy 420 297) (xy 0 297)
+        )
+      )
+    )
             (gr_line (start 53 147.5) (end 147 147.5) (angle 90) (layer Edge.Cuts) (width 0.15))
 (gr_line (start 147.5 147) (end 147.5 53) (angle 90) (layer Edge.Cuts) (width 0.15))

Commit message: Add ergogen logo
Parts:
- added LOGO1: , ceoloide:ergogen_logo, F.Cu at (100.0, 69.0)
- added LOGO10: , ceoloide:ergogen_logo, F.Cu at (197.0, 127.5)
- added LOGO2: , ceoloide:ergogen_logo, F.Cu at (235.0, 69.0)
- added LOGO3: , ceoloide:ergogen_logo, F.Cu at (100.0, 100.0)
- added LOGO4: , ceoloide:ergogen_logo, F.Cu at (235.0, 100.0)
- added LOGO5: , ceoloide:ergogen_logo, F.Cu at (100.0, 127.5)
- added LOGO6: , ceoloide:ergogen_logo, F.Cu at (235.0, 127.5)
- added LOGO7: , ceoloide:ergogen_logo, F.Cu at (119.0, 127.5)
- added LOGO8: , ceoloide:ergogen_logo, F.Cu at (216.0, 127.5)
- added LOGO9: , ceoloide:ergogen_logo, F.Cu at (138.0, 127.5)

Commit message: Updgrade to KiCad 8 PCB template
Other:
- net class Default removed
