File: pcbs/mx_demo.kicad_pcb (KiCad board)
At the start: 2 copper layers, 230 x 95 mm, 88 parts

Commit message: Update assets
Parts:
- moved D1 1.00 mm to (53.8, 144.7)
- moved D10 1.00 mm to (72.8, 68.7)
- moved D11 1.00 mm to (264.8, 144.7)
- moved D12 1.00 mm to (264.8, 125.7)
- moved D13 1.00 mm to (264.8, 106.7)
- moved D14 1.00 mm to (264.8, 87.7)
- moved D15 1.00 mm to (264.8, 68.7)
- moved D16 1.00 mm to (245.8, 144.7)
- moved D17 1.00 mm to (245.8, 125.7)
- moved D18 1.00 mm to (245.8, 106.7)
- moved D19 1.00 mm to (245.8, 87.7)
- moved D2 1.00 mm to (53.8, 125.7)
- moved D20 1.00 mm to (245.8, 68.7)
- moved D21 1.00 mm to (70.2, 144.7)
- moved D22 1.00 mm to (70.2, 125.7)
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Connections:
- S19 pad : (no net) -> LED_3
- S20 pad : (no net) -> LED_3
